Commit message: z_drive: updated rviz

File: z_drive/urdf/z_drive.urdf (robot description, URDF)
Before this commit: robot z_drive_system, 6 links, 5 joints
Links:
- link base_link: geometry 
- link port_prop: geometry visual cylinder length=0.0508 radius=0.0762
- link port_thruster: geometry collision box size=.1778 0.0762 0.127; visual box size=.1778 0.0762 0.127
- link starboard_prop: geometry visual cylinder length=0.0508 radius=0.0762
- link starboard_thruster: geometry collision box size=.1778 0.0762 0.127; visual box size=.1778 0.0762 0.127
- link z_drive_base: geometry visual box size=1.778 .889 .4064
Joints:
- joint port_servo: origin xyz=-.7239 .3048 0 rpy=0 0 0 -> xyz=-.7239 .3048 -0.254 rpy=3.14159 0 0
- joint starboard_servo: origin xyz=-.7239 -.3048 0 rpy=0 0 0 -> xyz=-.7239 -.3048 -0.254 rpy=3.14159 0 0

Commit message: boatsim: updated the simulation with darsens firctional forces

File: z_drive/urdf/z_drive.urdf (robot description, URDF)
Before this commit: robot z_drive, 6 links, 5 joints
Joints:
- removed joint port_thruster_to_prop
- removed joint starboard_thruster_to_prop
- added joint port_housing_to_prop: type prismatic, parent port_thruster, child port_prop, origin xyz=0 0 0 rpy=0 0 0, axis -1 0 0, limit lower=0 upper=1 effort=1 velocity=1
- added joint starboard_housing_to_prop: type prismatic, parent starboard_thruster, child starboard_prop, origin xyz=0 0 0 rpy=0 0 0, axis -1 0 0, limit lower=0 upper=1 effort=1 velocity=1
