Commit message: lidar test

File: propagator_description/robots/propagator_description.urdf (robot description, URDF)
Before this commit: robot propagator_description, 7 links, 6 joints
Joints:
- joint lidar_servo: origin xyz=0.645299789819263 -0.0669769690222898 0.27477134491897 rpy=-2.94943335198801 3.24078283203981E-05 1.57062975690281 -> xyz=0.645299789819263 -0.0669769690222898 0.27477134491897 rpy=0 0 0

Commit message: Lidar servo moving

File: propagator_description/robots/propagator_description.urdf (robot description, URDF)
Before this commit: robot propagator_description, 7 links, 6 joints
Joints:
- joint lidar_servo: axis 0 0 0 -> 0 1 0; limit (none) -> lower=0 upper=6.2832 effort=6 velocity=6.5973; type fixed -> revolute

Commit message: Fixing tf

File: propagator_description/robots/propagator_description.urdf (robot description, URDF)
Before this commit: robot propagator_description, 7 links, 6 joints
Joints:
- joint lidar_servo: origin xyz=0.645299789819263 -0.0669769690222898 0.27477134491897 rpy=0 0 0 -> xyz=0.645299789819263 -0.0669769690222898 0.27477134491897 rpy=0 0 3.14159

Commit message: Made motors.launch which remaps stm imu

File: propagator_description/robots/propagator_description.urdf (robot description, URDF)
Before this commit: robot propagator_description, 7 links, 6 joints
Joints:
- joint lidar_servo: limit lower=0 upper=6.2832 effort=6 velocity=6.5973 -> lower=0 upper=6.2832 effort=6 velocity=100
